Commit message: vision algorithm

File: cir_project/cirp_wam_description/xacro/iri_wam.urdf.xacro (robot description, xacro)
@@ -28,5 +28,5 @@
     <parent link="world"/>
     <child  link="${robot_name}_link_footprint"/>
-    <origin xyz="0 0 0" rpy="0 0 0" />
+    <origin xyz="0 0 0.72" rpy="0 0 0" />
   </joint>
   <xacro:wambase prefix="${robot_name}"/>
